Commit message: 0417

File: robot/urdf/h1.urdf (robot description, URDF)
Before this commit: robot h1_description, 22 links, 21 joints
Links:
- added link d435_left_imager_link; collision sphere radius=0.001; visual sphere radius=0.001
- added link d435_rgb_module_link; collision sphere radius=0.001; visual sphere radius=0.001
- added link mid360_link; collision sphere radius=0.001; visual sphere radius=0.001
- link left_ankle_link: mass 0.552448 -> 0.474; geometry collision box size=0.28 0.03 0.024; visual mesh filename=package://h1_description/meshes/left_ankle_link.dae
- link left_elbow_link: mass 0.669 -> 0.723; geometry collision cylinder length=0.09 radius=0.03; visual mesh filename=package://h1_description/meshes/left_elbow_link.dae
- link left_hip_pitch_link: geometry collision cylinder length=0.2 radius=0.05; visual mesh filename=package://h1_description/meshes/left_hip_pitch_link.dae
- link left_hip_roll_link: geometry collision cylinder length=0.01 radius=0.02; visual mesh filename=package://h1_description/meshes/left_hip_roll_link.dae
- link left_hip_yaw_link: geometry collision cylinder length=0.02 radius=0.01; visual mesh filename=package://h1_description/meshes/left_hip_yaw_link.dae
- link left_knee_link: geometry collision cylinder length=0.2 radius=0.05; visual mesh filename=package://h1_description/meshes/left_knee_link.dae
- link left_shoulder_pitch_link: geometry collision cylinder length=0.04 radius=0.03; visual mesh filename=package://h1_description/meshes/left_shoulder_pitch_link.dae
- link left_shoulder_roll_link: geometry collision cylinder length=0.01 radius=0.04; visual mesh filename=package://h1_description/meshes/left_shoulder_roll_link.dae
- link left_shoulder_yaw_link: geometry collision cylinder length=0.01 radius=0.04; visual mesh filename=package://h1_description/meshes/left_shoulder_yaw_link.dae
- link logo_link: geometry visual mesh filename=package://h1_description/meshes/logo_link.dae
- link pelvis: geometry collision sphere radius=0.05; visual mesh filename=package://h1_description/meshes/pelvis.dae
- link right_ankle_link: mass 0.552448 -> 0.474; geometry collision box size=0.28 0.03 0.024; visual mesh filename=package://h1_description/meshes/right_ankle_link.dae
- link right_elbow_link: mass 0.669 -> 0.723; geometry collision cylinder length=0.09 radius=0.03; visual mesh filename=package://h1_description/meshes/right_elbow_link.dae
- link right_hip_pitch_link: geometry collision cylinder length=0.2 radius=0.05; visual mesh filename=package://h1_description/meshes/right_hip_pitch_link.dae
- link right_hip_roll_link: geometry collision cylinder length=0.01 radius=0.02; visual mesh filename=package://h1_description/meshes/right_hip_roll_link.dae
- link right_hip_yaw_link: geometry collision cylinder length=0.02 radius=0.01; visual mesh filename=package://h1_description/meshes/right_hip_yaw_link.dae
- link right_knee_link: geometry collision cylinder length=0.2 radius=0.05; visual mesh filename=package://h1_description/meshes/right_knee_link.dae
- link right_shoulder_pitch_link: geometry collision cylinder length=0.04 radius=0.03; visual mesh filename=package://h1_description/meshes/right_shoulder_pitch_link.d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
- link right_shoulder_roll_link: geometry collision cylinder length=0.01 radius=0.04; visual mesh filename=package://h1_description/meshes/right_shoulder_roll_link.dae
- link right_shoulder_yaw_link: geometry collision cylinder length=0.01 radius=0.04; visual mesh filename=package://h1_description/meshes/right_shoulder_yaw_link.dae
- link torso_link: geometry collision box size=0.08 0.16 0.1; visual mesh filename=package://h1_description/meshes/torso_link.dae
Joints:
- added joint d435_left_imager_joint: type fixed, parent torso_link, child d435_left_imager_link, origin xyz=0.10848474394 0.0175 0.69317107367 rpy=-2.45735 0 -1.57080, axis 0 0 0
- added joint d435_rgb_module_joint: type fixed, parent torso_link, child d435_rgb_module_link, origin xyz=0.10848474394 0.0325 0.69317107367 rpy=-2.45735 0 -1.57080, axis 0 0 0
- added joint mid360_joint: type fixed, parent torso_link, child mid360_link, origin xyz=0.04729990180 0 0.67492878653 rpy=0 0.243124 0, axis 0 0 0
- joint left_elbow_joint: type fixed -> revolute
- joint left_hip_pitch_joint: limit lower=-1.57 upper=1.57 effort=200 velocity=23 -> lower=-3.14 upper=2.53 effort=200 velocity=23
- joint left_shoulder_pitch_joint: type fixed -> revolute
- joint left_shoulder_roll_joint: type fixed -> revolute
- joint left_shoulder_yaw_joint: type fixed -> revolute
- joint right_elbow_joint: type fixed -> revolute
- joint right_hip_pitch_joint: limit lower=-1.57 upper=1.57 effort=200 velocity=23 -> lower=-3.14 upper=2.53 effort=200 velocity=23
- joint right_shoulder_pitch_joint: type fixed -> revolute
- joint right_shoulder_roll_joint: type fixed -> revolute
- joint right_shoulder_yaw_joint: type fixed -> revolute
- joint torso_joint: type fixed -> revolute
